File: MJ65.kicad_pcb (KiCad board)
At the start: 2 copper layers, 285.7 x 120 mm, 230 parts, among them J0_0 Conn_01x02_Female, J1_0 Conn_01x02_Female, J2_0 Conn_01x02_Female, J3_0 Conn_01x02_Female, J4_0 Conn_01x02_Female, SW0_1 SW_Push, SW0_10 SW_Push, SW0_11 SW_Push, SW0_12 SW_Push, SW0_13 SW_Push, SW0_14 SW_Push, SW0_15 SW_Push, SW0_2 SW_Push, SW0_3 SW_Push, SW0_4 SW_Push, SW0_5 SW_Push, SW0_6 SW_Push, SW0_7 SW_Push, SW0_8 SW_Push, SW0_9 SW_Push, SW1_1 SW_Push, SW1_10 SW_Push, SW1_11 SW_Push, SW1_12 SW_Push, SW1_13 SW_Push, SW1_14 SW_Push, SW1_15 SW_Push, SW1_2 SW_Push, SW1_3 SW_Push, SW1_4 SW_Push, SW1_5 SW_Push, SW1_6 SW_Push, SW1_7 SW_Push, SW1_8 SW_Push, SW1_9 SW_Push, SW2_1 SW_Push, SW2_10 SW_Push, SW2_11 SW_Push, SW2_12 SW_Push, SW2_13 SW_Push, SW2_14 SW_Push, SW2_15 SW_Push, SW2_15_USEnt0 SW_Push, SW2_2 SW_Push, SW2_3 SW_Push, SW2_4 SW_Push, SW2_5 SW_Push, SW2_6 SW_Push, SW2_7 SW_Push, SW2_8 SW_Push, SW2_9 SW_Push, SW3_1 SW_Push, SW3_10 SW_Push, SW3_11 SW_Push, SW3_12 SW_Push, SW3_13 SW_Push, SW3_14 SW_Push, SW3_15 SW_Push, SW3_15_USSft0 SW_Push, SW3_2 SW_Push, SW3_3 SW_Push, SW3_4 SW_Push, SW3_5 SW_Push, SW3_6 SW_Push, SW3_7 SW_Push, SW3_8 SW_Push, SW3_9 SW_Push, SW4_1 SW_Push, SW4_10 SW_Push, SW4_10_USCmd0 SW_Push, SW4_11 SW_Push, SW4_12 SW_Push, SW4_13 SW_Push, SW4_13_AppL0 SW_Push, SW4_14 SW_Push, SW4_15 SW_Push, SW4_15_AppR0 SW_Push, SW4_2 SW_Push, SW4_3 SW_Push, SW4_4 SW_Push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

Commit message: Fix some route
Parts:
- SW2_15_USEnt0: footprint UniversalKeySwitch:Triple_PCB_225H-v-flip -> UniversalKeySwitch:Triple_PCB_225H
- turned SW2_15_USEnt0 to 0 degrees
Routing:
- net GND: track 0.00 -> 1364.2 mm
- net /R4: track 0.00 -> 583.9 mm
- net /R3: track 0.00 -> 472.8 mm
- net /C15: track 0.00 -> 451.8 mm, vias 0 -> 1
- net /C13: track 0.00 -> 444.4 mm, vias 0 -> 2
- net /R2: track 0.00 -> 408.2 mm
- net /C14: track 0.00 -> 407.6 mm
- net /R1: track 0.00 -> 357.4 mm
- net /C9: track 0.00 -> 343.5 mm, vias 0 -> 2
- net /C10: track 0.00 -> 327.8 mm
- net /C12: track 0.00 -> 317.1 mm
- net /C11: track 0.00 -> 314.3 mm, vias 0 -> 2
- net /R0: track 0.00 -> 273.1 mm
- net /C8: track 0.00 -> 237.9 mm, vias 0 -> 1
- net /C6: track 0.00 -> 230.4 mm, vias 0 -> 1
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
Commit message: Add GND filling
Routing:
- net /R2: track 408.2 -> 420.5 mm
- net /C9: track 343.5 -> 353.5 mm
- net /C10: track 327.8 -> 337.2 mm
- net /C14: track 407.6 -> 413.1 mm
- net /R4: track 583.9 -> 589.1 mm
- net /R1: track 357.4 -> 361.6 mm
- net /R3: track 472.8 -> 476.6 mm
- net /C2: track 119.5 -> 123.1 mm
- net /C12: track 317.1 -> 320.7 mm
- net /C13: track 444.4 -> 447.2 mm
- net Net-(D2_0-Pad2): track 21.9 -> 24.7 mm
- net /C6: track 230.4 -> 232.1 mm
- net /C11: track 314.3 -> 316.1 mm
- net /R0: track 273.1 -> 272.0 mm
- net /C7: track 216.6 -> 217.6 mm
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- added copper zone on B.Cu, net GND
- added copper zone on F.Cu, net GND

Commit message: Tweak routes for larger GND filling
Other:
- rule pad_to_mask_clearance: 0.051 -> 0.1
Changed lines of the file:
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@@
     (pad_size 4.4 4.4)
     (pad_drill 2.2)
-    (pad_to_mask_clearance 0.051)
+    (pad_to_mask_clearance 0.1)
     (solder_mask_min_width 0.25)
+    (pad_to_paste_clearance 0.1)
     (aux_axis_origin 0 0)
     (visible_elements FEFFFF7F)
     (pcbplotparams
       (layerselection 0x010fc_ffffffff)
-      (usegerberextensions false)
+      (usegerberextensions true)
       (usegerberattributes false)
       (usegerberadvancedattributes false)
@@
       (outputformat 1)
       (mirror false)
-      (drillshape 1)
+      (drillshape 0)
       (scaleselection 1)
-      (outputdirectory ""))
+      (outputdirectory "gerb/"))
   )
   (net 0 "")
