File: MJ65.kicad_pcb (KiCad board)
At the start: 2 copper layers, 285.7 x 120 mm, 230 parts, among them J0_0 Conn_01x02_Female, J1_0 Conn_01x02_Female, J2_0 Conn_01x02_Female, J3_0 Conn_01x02_Female, J4_0 Conn_01x02_Female, SW0_1 SW_Push, SW0_10 SW_Push, SW0_11 SW_Push, SW0_12 SW_Push, SW0_13 SW_Push, SW0_14 SW_Push, SW0_15 SW_Push, SW0_2 SW_Push, SW0_3 SW_Push, SW0_4 SW_Push, SW0_5 SW_Push, SW0_6 SW_Push, SW0_7 SW_Push, SW0_8 SW_Push, SW0_9 SW_Push, SW1_1 SW_Push, SW1_10 SW_Push, SW1_11 SW_Push, SW1_12 SW_Push, SW1_13 SW_Push, SW1_14 SW_Push, SW1_15 SW_Push, SW1_2 SW_Push, SW1_3 SW_Push, SW1_4 SW_Push, SW1_5 SW_Push, SW1_6 SW_Push, SW1_7 SW_Push, SW1_8 SW_Push, SW1_9 SW_Push, SW2_1 SW_Push, SW2_10 SW_Push, SW2_11 SW_Push, SW2_12 SW_Push, SW2_13 SW_Push, SW2_14 SW_Push, SW2_15 SW_Push, SW2_15_USEnt0 SW_Push, SW2_2 SW_Push, SW2_3 SW_Push, SW2_4 SW_Push, SW2_5 SW_Push, SW2_6 SW_Push, SW2_7 SW_Push, SW2_8 SW_Push, SW2_9 SW_Push, SW3_1 SW_Push, SW3_10 SW_Push, SW3_11 SW_Push, SW3_12 SW_Push, SW3_13 SW_Push, SW3_14 SW_Push, SW3_15 SW_Push, SW3_15_USSft0 SW_Push, SW3_2 SW_Push, SW3_3 SW_Push, SW3_4 SW_Push, SW3_5 SW_Push, SW3_6 SW_Push, SW3_7 SW_Push, SW3_8 SW_Push, SW3_9 SW_Push, SW4_1 SW_Push, SW4_10 SW_Push, SW4_10_USCmd0 SW_Push, SW4_11 SW_Push, SW4_12 SW_Push, SW4_13 SW_Push, SW4_13_AppL0 SW_Push, SW4_14 SW_Push, SW4_15 SW_Push, SW4_15_AppR0 SW_Push, SW4_2 SW_Push, SW4_3 SW_Push, SW4_4 SW_Push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

Commit message: Change footprint library to open source
Parts:
- D0_0, D0_1, D0_10, D0_11, D0_12, D0_13, D0_14, D0_15, D0_2, D0_3, D0_4, D0_5, D0_6, D0_7, D0_8, D0_9, D1_0, D1_1, D1_10, D1_11, D1_12, D1_13, D1_14, D1_15, D1_2, D1_3, D1_4, D1_5, D1_6, D1_7, D1_8, D1_9, D2_0, D2_1, D2_10, D2_11, D2_12, D2_13, D2_14, D2_15, D2_2, D2_3, D2_4, D2_5, D2_6, D2_7, D2_8, D2_9, D3_0, D3_1, D3_10, D3_11, D3_12, D3_13, D3_14, D3_15, D3_2, D3_3, D3_4, D3_5, D3_6, D3_7, D3_8, D3_9, D4_0, D4_1, D4_10, D4_11, D4_12, D4_13, D4_14, D4_15, D4_2, D4_3, D4_4, D4_5, D4_6, D4_7, D4_8, D4_9: footprint Keebio-Parts:Diode-dual -> Keebio-Parts (fork):Diode-dual
- J0_0, J1_0, J2_0, J3_0, J4_0, SW1_14, SW2_14, SW3_13, SW3_14, SW4_13, SW4_9: footprint UniversalKeySwitch:Triple_PCB_100H-External-Switch-Pad -> Keebio-Parts (fork):Triple_PCB_100H-External-Switch-Pad
- SW0_1, SW0_10, SW0_11, SW0_12, SW0_13, SW0_14, SW0_15, SW0_2, SW0_3, SW0_4, SW0_5, SW0_6, SW0_7, SW0_8, SW0_9, SW1_10, SW1_11, SW1_12, SW1_13, SW1_2, SW1_3, SW1_4, SW1_5, SW1_6, SW1_7, SW1_8, SW1_9, SW2_10, SW2_11, SW2_12, SW2_13, SW2_2, SW2_3, SW2_4, SW2_5, SW2_6, SW2_7, SW2_8, SW2_9, SW3_10, SW3_11, SW3_12, SW3_2, SW3_3, SW3_4, SW3_5, SW3_6, SW3_7, SW3_8, SW3_9, SW4_10_USCmd0, SW4_11, SW4_13_AppL0, SW4_14, SW4_15_AppR0, SW4_2, SW4_6: footprint UniversalKeySwitch:Triple_PCB_100H -> Keebio-Parts (fork):Triple_PCB_100H
- SW1_1, SW1_15, SW4_1, SW4_12, SW4_15: footprint UniversalKeySwitch:Triple_PCB_150H -> Keebio-Parts (fork):Triple_PCB_150H
- SW2_1, SW3_15, SW4_5, SW4_7: footprint UniversalKeySwitch:Triple_PCB_175H -> Keebio-Parts (fork):Triple_PCB_175H
- SW2_15: footprint UniversalKeySwitch:Triple_PCB_200V -> Keebio-Parts (fork):Triple_PCB_200V
- SW2_15_USEnt0, SW3_1: footprint UniversalKeySwitch:Triple_PCB_225H -> Keebio-Parts (fork):Triple_PCB_225H
- SW3_15_USSft0: footprint UniversalKeySwitch:Triple_PCB_275H-v-flip -> Keebio-Parts (fork):Triple_PCB_275H-v-flip
- SW4_10, SW4_3, SW4_4, SW4_8: footprint UniversalKeySwitch:Triple_PCB_125H -> Keebio-Parts (fork):Triple_PCB_125H
- SW4_6_USSp0: footprint UniversalKeySwitch:Triple_PCB_625H-v-flip -> Keebio-Parts (fork):Triple_PCB_625H-v-flip

Commit message: Tweak some wiring & ready to submission
Routing:
- net /R3: track 476.6 -> 479.5 mm
- net /R0: track 272.0 -> 272.6 mm

Commit message: Remove unneeded wiring among GND mount holes
Routing:
- net GND: track 1363.7 -> 63.5 mm

Commit message: Fix duplicated SW4_13
Parts:
- removed G***: LOGO, logo:logo10x10
- removed J0_0, J1_0, J2_0, J3_0, J4_0: Conn_01x02_Female, Keebio-Parts (fork):Triple_PCB_100H-External-Switch-Pad
- removed SW4_13_AppL0: SW_Push, Keebio-Parts (fork):Triple_PCB_100H
- added SW0_0: SW_Push, Keebio-Parts (fork):Triple_PCB_100H-External-Switch-Pad, F.Cu at (57.1, 10.5)
- added SW1_0: SW_Push, Keebio-Parts (fork):Triple_PCB_100H-External-Switch-Pad, F.Cu at (76.2, 10.5)
- added SW2_0: SW_Push, Keebio-Parts (fork):Triple_PCB_100H-External-Switch-Pad, F.Cu at (95.2, 10.5)
- added SW3_0: SW_Push, Keebio-Parts (fork):Triple_PCB_100H-External-Switch-Pad, F.Cu at (114.3, 10.5)
- added SW4_0: SW_Push, Keebio-Parts (fork):Triple_PCB_100H-External-Switch-Pad, F.Cu at (142.8, 10.5)
- added SW4_12_AppL0: SW_Push, Keebio-Parts (fork):Triple_PCB_100H, F.Cu at (238.0, 110.5)
Connections:
- U0 pad 1: Net-(U0-Pad1) -> (no net)
- U0 pad 11: Net-(U0-Pad11) -> (no net)
- U0 pad 15: Net-(U0-Pad15) -> (no net)
- U0 pad 2: Net-(U0-Pad2) -> (no net)
- U0 pad 24: Net-(U0-Pad24) -> (no net)
- U0 pad 3: Net-(U0-Pad3) -> (no net)
- U0 pad 31: Net-(U0-Pad31) -> (no net)
- U0 pad 33: Net-(U0-Pad33) -> (no net)
- U0 pad 4: Net-(U0-Pad4) -> (no net)
Routing:
- net Net-(D4_13-Pad2): track 161.9 -> 14.1 mm
- net /C13: track 447.2 -> 398.7 mm, vias 2 -> 1
- net /C12: track 320.7 -> 345.3 mm
- net Net-(D4_12-Pad2): track 7.57 -> 25.4 mm
