File: MJ65.sch (KiCad schematic (older format))
At the start: 167 parts, among them J0_0 Conn_01x02_Female, J1_0 Conn_01x02_Female, J2_0 Conn_01x02_Female, J3_0 Conn_01x02_Female, J4_0 Conn_01x02_Female, SW0_1 SW_Push, SW0_10 SW_Push, SW0_11 SW_Push, SW0_12 SW_Push, SW0_13 SW_Push, SW0_14 SW_Push, SW0_15 SW_Push, SW0_2 SW_Push, SW0_3 SW_Push, SW0_4 SW_Push, SW0_5 SW_Push, SW0_6 SW_Push, SW0_7 SW_Push, SW0_8 SW_Push, SW0_9 SW_Push, SW1_1 SW_Push, SW1_10 SW_Push, SW1_11 SW_Push, SW1_12 SW_Push, SW1_13 SW_Push, SW1_14 SW_Push, SW1_15 SW_Push, SW1_2 SW_Push, SW1_3 SW_Push, SW1_4 SW_Push, SW1_5 SW_Push, SW1_6 SW_Push, SW1_7 SW_Push, SW1_8 SW_Push, SW1_9 SW_Push, SW2_1 SW_Push, SW2_10 SW_Push, SW2_11 SW_Push, SW2_12 SW_Push, SW2_13 SW_Push, SW2_14 SW_Push, SW2_15 SW_Push, SW2_15_USEnt0 SW_Push, SW2_2 SW_Push, SW2_3 SW_Push, SW2_4 SW_Push, SW2_5 SW_Push, SW2_6 SW_Push, SW2_7 SW_Push, SW2_8 SW_Push, SW2_9 SW_Push, SW3_1 SW_Push, SW3_10 SW_Push, SW3_11 SW_Push, SW3_12 SW_Push, SW3_13 SW_Push, SW3_14 SW_Push, SW3_15 SW_Push, SW3_15_USSft0 SW_Push, SW3_2 SW_Push, SW3_3 SW_Push, SW3_4 SW_Push, SW3_5 SW_Push, SW3_6 SW_Push, SW3_7 SW_Push, SW3_8 SW_Push, SW3_9 SW_Push, SW4_1 SW_Push, SW4_10 SW_Push, SW4_10_USCmd0 SW_Push, SW4_11 SW_Push, SW4_12 SW_Push, SW4_13 SW_Push, SW4_13_AppL0 SW_Push, SW4_14 SW_Push, SW4_15 SW_Push, SW4_15_AppR0 SW_Push, SW4_2 SW_Push, SW4_3 SW_Push, SW4_4 SW_Push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

Commit message: Change footprint library to open source
Parts:
- D0_0, D0_1, D0_10, D0_11, D0_12, D0_13, D0_14, D0_15, D0_2, D0_3, D0_4, D0_5, D0_6, D0_7, D0_8, D0_9, D1_0, D1_1, D1_10, D1_11, D1_12, D1_13, D1_14, D1_15, D1_2, D1_3, D1_4, D1_5, D1_6, D1_7, D1_8, D1_9, D2_0, D2_1, D2_10, D2_11, D2_12, D2_13, D2_14, D2_15, D2_2, D2_3, D2_4, D2_5, D2_6, D2_7, D2_8, D2_9, D3_0, D3_1, D3_10, D3_11, D3_12, D3_13, D3_14, D3_15, D3_2, D3_3, D3_4, D3_5, D3_6, D3_7, D3_8, D3_9, D4_0, D4_1, D4_10, D4_11, D4_12, D4_13, D4_14, D4_15, D4_2, D4_3, D4_4, D4_5, D4_6, D4_7, D4_8, D4_9: footprint Keebio-Parts:Diode-dual -> Keebio-Parts (fork):Diode-dual
- J0_0, J1_0, J2_0, J3_0, J4_0, SW1_14, SW2_14, SW3_13, SW3_14, SW4_13, SW4_9: footprint UniversalKeySwitch:Triple_PCB_100H-External-Switch-Pad -> Keebio-Parts (fork):Triple_PCB_100H-External-Switch-Pad
- SW0_1, SW0_10, SW0_11, SW0_12, SW0_13, SW0_14, SW0_15, SW0_2, SW0_3, SW0_4, SW0_5, SW0_6, SW0_7, SW0_8, SW0_9, SW1_10, SW1_11, SW1_12, SW1_13, SW1_2, SW1_3, SW1_4, SW1_5, SW1_6, SW1_7, SW1_8, SW1_9, SW2_10, SW2_11, SW2_12, SW2_13, SW2_2, SW2_3, SW2_4, SW2_5, SW2_6, SW2_7, SW2_8, SW2_9, SW3_10, SW3_11, SW3_12, SW3_2, SW3_3, SW3_4, SW3_5, SW3_6, SW3_7, SW3_8, SW3_9, SW4_10_USCmd0, SW4_11, SW4_13_AppL0, SW4_14, SW4_15_AppR0, SW4_2, SW4_6: footprint UniversalKeySwitch:Triple_PCB_100H -> Keebio-Parts (fork):Triple_PCB_100H
- SW1_1, SW1_15, SW4_1, SW4_12, SW4_15: footprint UniversalKeySwitch:Triple_PCB_150H -> Keebio-Parts (fork):Triple_PCB_150H
- SW2_1, SW3_15, SW4_5, SW4_7: footprint UniversalKeySwitch:Triple_PCB_175H -> Keebio-Parts (fork):Triple_PCB_175H
- SW2_15: footprint UniversalKeySwitch:Triple_PCB_200V -> Keebio-Parts (fork):Triple_PCB_200V
- SW2_15_USEnt0: footprint UniversalKeySwitch:Triple_PCB_225H-v-flip -> Keebio-Parts (fork):Triple_PCB_225H
- SW3_1: footprint UniversalKeySwitch:Triple_PCB_225H -> Keebio-Parts (fork):Triple_PCB_225H
- SW3_15_USSft0: footprint UniversalKeySwitch:Triple_PCB_275H-v-flip -> Keebio-Parts (fork):Triple_PCB_275H-v-flip
- SW4_10, SW4_3, SW4_4, SW4_8: footprint UniversalKeySwitch:Triple_PCB_125H -> Keebio-Parts (fork):Triple_PCB_125H
- SW4_6_USSp0: footprint UniversalKeySwitch:Triple_PCB_625H-v-flip -> Keebio-Parts (fork):Triple_PCB_625H-v-flip

Commit message: Fix duplicated SW4_13
Parts:
- removed J0_0, J1_0, J2_0, J3_0, J4_0: Conn_01x02_Female, Keebio-Parts (fork):Triple_PCB_100H-External-Switch-Pad, symbol Connector:Conn_01x02_Female
- removed SW4_13_AppL0: SW_Push, Keebio-Parts (fork):Triple_PCB_100H, symbol Switch:SW_Push
- added SW0_0, SW1_0, SW2_0, SW3_0, SW4_0: SW_Push, Keebio-Parts (fork):Triple_PCB_100H-External-Switch-Pad, symbol Switch:SW_Push
- added SW4_12_AppL0: SW_Push, Keebio-Parts (fork):Triple_PCB_100H, symbol Switch:SW_Push
Connections:
- net C0: now also SW0_0.1, SW1_0.1, SW2_0.1, SW3_0.1, SW4_0.1
- net C12: now also SW4_12_AppL0.2
- net at D4_0.2 (A): now also SW4_0.2
- net at D3_0.2 (A): now also SW3_0.2
- net at D2_0.2 (A): now also SW2_0.2
- net at D1_0.2 (A): now also SW1_0.2
- net at D0_0.2 (A): now also SW0_0.2
- net at D4_12.2 (A), SW4_12.1: now also SW4_12_AppL0.1
Other:
- moved on the sheet: D0_0, D1_0, D2_0, D3_0, D4_0
Changed lines of the file:
@@
 L Device:D D4_0
 U 1 1 5C9DD1BC
-P 4650 4950
-F 0 "D4_0" V 4604 5078 50  0000 L CNN
-F 1 "DIODE" V 4695 5078 50  0000 L CNN
-F 2 "Keebio-Parts (fork):Diode-dual" H 4650 4950 50  0001 C CNN
-F 3 "~" H 4650 4950 50  0001 C CNN
-	1    4650 4950
+P 4750 4950
+F 0 "D4_0" V 4704 5078 50  0000 L CNN
+F 1 "DIODE" V 4795 5078 50  0000 L CNN
+F 2 "Keebio-Parts (fork):Diode-dual" H 4750 4950 50  0001 C CNN
+F 3 "~" H 4750 4950 50  0001 C CNN
+	1    4750 4950
 	0    1    1    0
 $EndComp
@@
 L Device:D D3_0
 U 1 1 5CA06939
-P 4650 3750
-F 0 "D3_0" V 4604 3878 50  0000 L CNN
-F 1 "DIODE" V 4695 3878 50  0000 L CNN
-F 2 "Keebio-Parts (fork):Diode-dual" H 4650 3750 50  0001 C CNN
-F 3 "~" H 4650 3750 50  0001 C CNN
-	1    4650 3750
+P 4750 3750
+F 0 "D3_0" V 4704 3878 50  0000 L CNN
+F 1 "DIODE" V 4795 3878 50  0000 L CNN
+F 2 "Keebio-Parts (fork):Diode-dual" H 4750 3750 50  0001 C CNN
+F 3 "~" H 4750 3750 50  0001 C CNN
+	1    4750 3750
 	0    1    1    0
 $EndComp
@@
 L Device:D D2_0
 U 1 1 5CA1A1E0
-P 4650 2550
-F 0 "D2_0" V 4604 2678 50  0000 L CNN
-F 1 "DIODE" V 4695 2678 50  0000 L CNN
-F 2 "Keebio-Parts (fork):Diode-dual" H 4650 2550 50  0001 C CNN
-F 3 "~" H 4650 2550 50  0001 C CNN
-	1    4650 2550
+P 4750 2550
+F 0 "D2_0" V 4704 2678 50  0000 L CNN
+F 1 "DIODE" V 4795 2678 50  0000 L CNN
+F 2 "Keebio-Parts (fork):Diode-dual" H 4750 2550 50  0001 C CNN
+F 3 "~" H 4750 2550 50  0001 C CNN
+	1    4750 2550
 	0    1    1    0
 $EndComp
@@
 L Device:D D1_0
 U 1 1 5CA2C5A4
-P 4650 1800
-F 0 "D1_0" V 4604 1928 50  0000 L CNN
-F 1 "DIODE" V 4695 1928 50  0000 L CNN
-F 2 "Keebio-Parts (fork):Diode-dual" H 4650 1800 50  0001 C CNN
-F 3 "~" H 4650 1800 50  0001 C CNN
-	1    4650 1800
+P 4750 1800
+F 0 "D1_0" V 4704 1928 50  0000 L CNN
+F 1 "DIODE" V 4795 1928 50  0000 L CNN
+F 2 "Keebio-Parts (fork):Diode-dual" H 4750 1800 50  0001 C CNN
+F 3 "~" H 4750 1800 50  0001 C CNN
+	1    4750 1800
 	0    1    1    0
 $EndComp
@@
 $EndComp
 $Comp
-L Connector:Conn_01x02_Female J4_0
-U 1 1 5C6C9FED
-P 4950 5300
-F 0 "J4_0" V 4797 5348 50  0000 L CNN
-F 1 "Conn_01x02_Female" V 4888 5348 50  0000 L CNN
-F 2 "Keebio-Parts (fork):Triple_PCB_100H-External-Switch-Pad" H 4950 5300 50  0001 C CNN
-F 3 "~" H 4950 5300 50  0001 C CNN
-	1    4950 5300
-	0    1    1    0
-$EndComp
-Wire Wire Line
-	4650 5100 4850 5100
-Wire Wire Line
-	4950 5100 5150 5100
-Connection ~ 5150 5100
-Wire Wire Line
-	5150 1200 5150 1950
-$Comp
-L Connector:Conn_01x02_Female J3_0
-U 1 1 5C77E4EE
-P 4950 4100
-F 0 "J3_0" V 4797 4148 50  0000 L CNN
-F 1 "Conn_01x02_Female" V 4888 4148 50  0000 L CNN
-F 2 "Keebio-Parts (fork):Triple_PCB_100H-External-Switch-Pad" H 4950 4100 50  0001 C CNN
-F 3 "~" H 4950 4100 50  0001 C CNN
-	1    4950 4100
-	0    1    1    0
-$EndComp
-$Comp
-L Connector:Conn_01x02_Female J2_0
-U 1 1 5C77F3E6
-P 4950 2900
-F 0 "J2_0" V 4797 2948 50  0000 L CNN
-F 1 "Conn_01x02_Female" V 4888 2948 50  0000 L CNN
-F 2 "Keebio-Parts (fork):Triple_PCB_100H-External-Switch-Pad" H 4950 2900 50  0001 C CNN
-F 3 "~" H 4950 2900 50  0001 C CNN
-	1    4950 2900
-	0    1    1    0
-$EndComp
-$Comp
-L Connector:Conn_01x02_Female J1_0
-U 1 1 5C77FF14
-P 4950 2150
-F 0 "J1_0" V 4797 2198 50  0000 L CNN
-F 1 "Conn_01x02_Female" V 4888 2198 50  0000 L CNN
-F 2 "Keebio-Parts (fork):Triple_PCB_100H-External-Switch-Pad" H 4950 2150 50  0001 C CNN
-F 3 "~" H 4950 2150 50  0001 C CNN
-	1    4950 2150
-	0    1    1    0
-$EndComp
-$Comp
-L Connector:Conn_01x02_Female J0_0
-U 1 1 5C780A51
-P 4950 1400
-F 0 "J0_0" V 4797 1448 50  0000 L CNN
-F 1 "Conn_01x02_Female" V 4888 1448 50  0000 L CNN
-F 2 "Keebio-Parts (fork):Triple_PCB_100H-External-Switch-Pad" H 4950 1400 50  0001 C CNN
-F 3 "~" H 4950 1400 50  0001 C CNN
-	1    4950 1400
-	0    1    1    0
-$EndComp
-Wire Wire Line
-	5150 1200 4950 1200
-Wire Wire Line
-	4850 1200 4650 1200
-Wire Wire Line
-	4950 1950 5150 1950
-Connection ~ 5150 1950
-Wire Wire Line
-	5150 1950 5150 2700
-Wire Wire Line
-	4850 1950 4650 1950
-Wire Wire Line
-	4950 2700 5150 2700
-Connection ~ 5150 2700
-Wire Wire Line
-	5150 2700 5150 3900
-Wire Wire Line
-	4850 2700 4650 2700
-Wire Wire Line
-	4950 3900 5150 3900
-Connection ~ 5150 3900
-Wire Wire Line
-	5150 3900 5150 5100
-Wire Wire Line
-	4850 3900 4650 3900
-$Comp
 L power:PWR_FLAG #FLG0101
 U 1 1 5C82F821
@@
 $EndComp
 Wire Wire Line
-	5150 5100 5150 5750
-Wire Wire Line
 	5850 5100 5850 5750
 Wire Wire Line
@@
 	12850 5100 12850 5750
 Wire Wire Line
-	13550 5100 13550 5750
-Wire Wire Line
-	14250 5100 14250 5500
+	13550 5100 13550 5500
 Wire Wire Line
 	14950 5100 14950 5750
@@
 	15250 3100 15250 2700
 Wire Wire Line
-	4100 800  4650 800
+	4100 800  4750 800
 $Comp
 L Device:D D0_0
 U 1 1 5C8D3C5F
-P 4650 1050
-F 0 "D0_0" V 4604 1129 50  0000 L CNN
-F 1 "D" V 4695 1129 50  0000 L CNN
-F 2 "Keebio-Parts (fork):Diode-dual" H 4650 1050 50  0001 C CNN
-F 3 "~" H 4650 1050 50  0001 C CNN
-	1    4650 1050
+P 4750 1050
+F 0 "D0_0" V 4704 1129 50  0000 L CNN
+F 1 "D" V 4795 1129 50  0000 L CNN
+F 2 "Keebio-Parts (fork):Diode-dual" H 4750 1050 50  0001 C CNN
+F 3 "~" H 4750 1050 50  0001 C CNN
+	1    4750 1050
 	0    1    1    0
 $EndComp
 Wire Wire Line
-	4650 900  4650 800
-Connection ~ 4650 800
-Wire Wire Line
-	4650 800  5450 800
+	4750 900  4750 800
+Connection ~ 4750 800
+Wire Wire Line
+	4750 800  5450 800
 Wire Wire Line
 	5450 900  5450 800
@@
 	15250 800  15250 900
 Wire Wire Line
-	4100 1550 4650 1550
-Wire Wire Line
-	4650 1650 4650 1550
-Connection ~ 4650 1550
-Wire Wire Line
-	4650 1550 5450 1550
+	4100 1550 4750 1550
+Wire Wire Line
+	4750 1650 4750 1550
+Connection ~ 4750 1550
+Wire Wire Line
+	4750 1550 5450 1550
 Wire Wire Line
 	5450 1650 5450 1550
@@
 	15250 1650 15250 1550
 Wire Wire Line
-	4100 2300 4650 2300
-Wire Wire Line
-	4650 2400 4650 2300
-Connection ~ 4650 2300
-Wire Wire Line
-	4650 2300 5450 2300
+	4100 2300 4750 2300
+Wire Wire Line
+	4750 2400 4750 2300
+Connection ~ 4750 2300
+Wire Wire Line
+	4750 2300 5450 2300
 Wire Wire Line
 	5450 2400 5450 2300
@@
 	15250 2400 15250 2300
 Wire Wire Line
-	4100 3500 4650 3500
-Wire Wire Line
-	4650 3600 4650 3500
-Connection ~ 4650 3500
-Wire Wire Line
-	4650 3500 5450 3500
+	4100 3500 4750 3500
+Wire Wire Line
+	4750 3600 4750 3500
+Connection ~ 4750 3500
+Wire Wire Line
+	4750 3500 5450 3500
 Wire Wire Line
 	5450 3600 5450 3500
@@
 	15250 3600 15250 3500
 Wire Wire Line
-	4100 4700 4650 4700
-Wire Wire Line
-	4650 4800 4650 4700
-Connection ~ 4650 4700
-Wire Wire Line
-	4650 4700 5450 4700
+	4100 4700 4750 4700
+Wire Wire Line
+	4750 4800 4750 4700
+Connection ~ 4750 4700
+Wire Wire Line
+	4750 4700 5450 4700
 Wire Wire Line
 	5450 4800 5450 4700
@@
 Connection ~ 8950 5100
 $Comp
-L Switch:SW_Push SW4_13_AppL0
-U 1 1 5D87C1DF
-P 14050 5500
-F 0 "SW4_13_AppL0" H 14050 5785 50  0000 C CNN
-F 1 "SW_Push" H 14050 5694 50  0000 C CNN
-F 2 "Keebio-Parts (fork):Triple_PCB_100H" H 14050 5700 50  0001 C CNN
-F 3 "" H 14050 5700 50  0001 C CNN
-	1    14050 5500
-	1    0    0    1
-$EndComp
-Connection ~ 14250 5500
-Wire Wire Line
-	14250 5500 14250 5750
-$Comp
 L Switch:SW_Push SW4_15_AppR0
 U 1 1 5D87D227
@@
 Connection ~ 15250 5100
 Wire Wire Line
-	13850 5500 13850 5100
-Connection ~ 13850 5100
+	14250 5100 14250 5750
+$Comp
+L Switch:SW_Push SW4_12_AppL0
+U 1 1 5C8721BD
+P 13350 5500
+F 0 "SW4_12_AppL0" H 13350 5785 50  0000 C CNN
+F 1 "SW_Push" H 13350 5694 50  0000 C CNN
+F 2 "Keebio-Parts (fork):Triple_PCB_100H" H 13350 5700 50  0001 C CNN
+F 3 "" H 13350 5700 50  0001 C CNN
+	1    13350 5500
+	1    0    0    1
+$EndComp
+Wire Wire Line
+	13150 5500 13150 5100
+$Comp
+L Switch:SW_Push SW0_0
+U 1 1 5C8A672D
+P 4950 1200
+F 0 "SW0_0" H 4950 1485 50  0000 C CNN
+F 1 "SW_Push" H 4950 1394 50  0000 C CNN
+F 2 "Keebio-Parts (fork):Triple_PCB_100H-External-Switch-Pad" H 4950 1400 50  0001 C CNN
+F 3 "" H 4950 1400 50  0001 C CNN
+	1    4950 1200
+	-1   0    0    -1
+$EndComp
+$Comp
+L Switch:SW_Push SW1_0
+U 1 1 5C95737E
+P 4950 1950
+F 0 "SW1_0" H 4950 2235 50  0000 C CNN
+F 1 "SW_Push" H 4950 2144 50  0000 C CNN
+F 2 "Keebio-Parts (fork):Triple_PCB_100H-External-Switch-Pad" H 4950 2150 50  0001 C CNN
+F 3 "" H 4950 2150 50  0001 C CNN
+	1    4950 1950
+	-1   0    0    -1
+$EndComp
+$Comp
+L Switch:SW_Push SW2_0
+U 1 1 5C9C51B4
+P 4950 2700
+F 0 "SW2_0" H 4950 2985 50  0000 C CNN
+F 1 "SW_Push" H 4950 2894 50  0000 C CNN
+F 2 "Keebio-Parts (fork):Triple_PCB_100H-External-Switch-Pad" H 4950 2900 50  0001 C CNN
+F 3 "" H 4950 2900 50  0001 C CNN
+	1    4950 2700
+	-1   0    0    -1
+$EndComp
+$Comp
+L Switch:SW_Push SW3_0
+U 1 1 5CA3226B
+P 4950 3900
+F 0 "SW3_0" H 4950 4185 50  0000 C CNN
+F 1 "SW_Push" H 4950 4094 50  0000 C CNN
+F 2 "Keebio-Parts (fork):Triple_PCB_100H-External-Switch-Pad" H 4950 4100 50  0001 C CNN
+F 3 "" H 4950 4100 50  0001 C CNN
+	1    4950 3900
+	-1   0    0    -1
+$EndComp
+$Comp
+L Switch:SW_Push SW4_0
+U 1 1 5CA9D2CE
+P 4950 5100
+F 0 "SW4_0" H 4950 5385 50  0000 C CNN
+F 1 "SW_Push" H 4950 5294 50  0000 C CNN
+F 2 "Keebio-Parts (fork):Triple_PCB_100H-External-Switch-Pad" H 4950 5300 50  0001 C CNN
+F 3 "" H 4950 5300 50  0001 C CNN
+	1    4950 5100
+	-1   0    0    -1
+$EndComp
+Connection ~ 5150 5100
+Wire Wire Line
+	5150 5100 5150 5750
+Connection ~ 5150 3900
+Wire Wire Line
+	5150 3900 5150 5100
+Connection ~ 5150 2700
+Wire Wire Line
+	5150 2700 5150 3900
+Wire Wire Line
+	5150 1200 5150 1950
+Connection ~ 5150 1950
+Wire Wire Line
+	5150 1950 5150 2700
+Connection ~ 13550 5500
+Wire Wire Line
+	13550 5500 13550 5750
 $EndSCHEMATC
